File: KICAD pcb/maibadge/maibadge_ver2.kicad_sch (KiCad schematic)
At the start: 22 parts, among them J1 Conn_01x04_Socket, SW1 SW_Push, SW2 SW_Push, SW3 SW_Push, SW4 SW_Push, U1 ESP32-S3-WROOM-1, U10 SK6812SIDE-A-RVS, U11 MPR121QR2, U2 AMS1117-3.3, U3 SK6812SIDE-A-RVS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

Commit message: fix: schematic and routing
Parts:
- removed U11: MPR121QR2, Maibadge_Howard:QFN-20_L3.0-W3.0-P0.40-BL, symbol amaibear:MPR121QR2
Connections:
- net MPR SDA is gone; now on net buzzer: U1.24 (IO47)
- net +5V: now also J1.4 (Pin_4); no longer J1.1 (Pin_1)
- net GND: now also J1.1 (Pin_1); no longer J1.4 (Pin_4)
- net buzzer: no longer U1.33 (IO40)
- net main led DIN: now also U1.8 (IO15); no longer U1.35 (IO42)
- net MPR SCL: no longer names the net of U1.25 (IO48)
Other:
- note removed: "(not using MPR121 as ESP32 has built-in capacitive touch)"
- note removed: "capacitive touch"
