File: KICAD pcb/maibadge/maibadge_ver2.kicad_sch (KiCad schematic)
At the start: 20 parts, among them J1 Conn_01x04_Socket, SW3 SW_Push, SW4 SW_Push, SW5 SW_Push, U1 ESP32-S3-WROOM-1, U10 SK6812SIDE-A-RVS, U11 MPR121QR2, U2 AMS1117-3.3, U3 SK6812SIDE-A-RVS, U4 SK6812SIDE-A-RVS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

Commit message: feat: maibadge cab v2
Connections:
- net USB_D+: now also J1.3 (Pin_3); no longer J1.2 (Pin_2)
- net USB_D-: now also J1.2 (Pin_2); no longer J1.3 (Pin_3)
Changed lines of the file:
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@@
+	(wire
+		(pts
+			(xy 144.78 120.65) (xy 156.21 120.65)
+		)
+		(stroke
+			(width 0)
+			(type default)
+		)
+	)
 	(wire
 		(pts
@@
 	(wire
 		(pts
-			(xy 144.78 120.65) (xy 156.21 120.65)
-		)
-		(stroke
-			(width 0)
-			(type default)
-		)
-	)
-	(wire
-		(pts
 			(xy 107.95 118.11) (xy 107.95 124.46)
 		)
@@
 		)
 	)
+	(polyline
+		(pts
+			(xy 76.2 19.05) (xy 76.2 176.53)
+		)
+		(stroke
+			(width 1)
+			(type default)
+		)
+	)
+	(wire
+		(pts
+			(xy 107.95 142.24) (xy 107.95 147.32)
+		)
+		(stroke
+			(width 0)
+			(type default)
+		)
+	)
+	(wire
+		(pts
+			(xy 199.39 46.99) (xy 199.39 41.91)
+		)
+		(stroke
+			(width 0)
+			(type default)
+		)
+	)
+	(wire
+		(pts
+			(xy 146.05 123.19) (xy 156.21 123.19)
+		)
+		(stroke
+			(width 0)
+			(type default)
+		)
+	)
+	(wire
+		(pts
+			(xy 196.85 58.42) (xy 196.85 60.96)
+		)
+		(stroke
+			(width 0)
+			(type default)
+		)
+	)
+	(wire
+		(pts
+			(xy 196.85 49.53) (xy 196.85 58.42)
+		)
+		(stroke
+			(width 0)
+			(type default)
+		)
+	)
+	(wire
+		(pts
+			(xy 31.75 147.32) (xy 39.37 147.32)
+		)
+		(stroke
+			(width 0)
+			(type default)
+		)
+	)
+	(wire
+		(pts
+			(xy 144.78 115.57) (xy 156.21 115.57)
+		)
+		(stroke
+			(width 0)
+			(type default)
+		)
+	)
+	(wire
+		(pts
+			(xy 107.95 147.32) (xy 120.65 147.32)
+		)
+		(stroke
+			(width 0)
+			(type default)
+		)
+	)
+	(wire
+		(pts
+			(xy 92.71 142.24) (xy 97.79 142.24)
+		)
+		(stroke
+			(width 0)
+			(type default)
+		)
+	)
+	(wire
+		(pts
+			(xy 107.95 124.46) (xy 116.84 124.46)
+		)
+		(stroke
+			(width 0)
+			(type default)
+		)
+	)
 	(wire
 		(pts
 			(xy 144.78 118.11) (xy 156.21 118.11)
-		)
-		(stroke
-			(width 0)
-			(type default)
-		)
-	)
-	(polyline
-		(pts
-			(xy 76.2 19.05) (xy 76.2 176.53)
-		)
-		(stroke
-			(width 1)
-			(type default)
-		)
-	)
-	(wire
-		(pts
-			(xy 107.95 142.24) (xy 107.95 147.32)
-		)
-		(stroke
-			(width 0)
-			(type default)
-		)
-	)
-	(wire
-		(pts
-			(xy 199.39 46.99) (xy 199.39 41.91)
-		)
-		(stroke
-			(width 0)
-			(type default)
-		)
-	)
-	(wire
-		(pts
-			(xy 146.05 123.19) (xy 156.21 123.19)
-		)
-		(stroke
-			(width 0)
-			(type default)
-		)
-	)
-	(wire
-		(pts
-			(xy 196.85 58.42) (xy 196.85 60.96)
-		)
-		(stroke
-			(width 0)
-			(type default)
-		)
-	)
-	(wire
-		(pts
-			(xy 196.85 49.53) (xy 196.85 58.42)
-		)
-		(stroke
-			(width 0)
-			(type default)
-		)
-	)
-	(wire
-		(pts
-			(xy 31.75 147.32) (xy 39.37 147.32)
-		)
-		(stroke
-			(width 0)
-			(type default)
-		)
-	)
-	(wire
-		(pts
-			(xy 144.78 115.57) (xy 156.21 115.57)
-		)
-		(stroke
-			(width 0)
-			(type default)
-		)
-	)
-	(wire
-		(pts
-			(xy 107.95 147.32) (xy 120.65 147.32)
-		)
-		(stroke
-			(width 0)
-			(type default)
-		)
-	)
-	(wire
-		(pts
-			(xy 92.71 142.24) (xy 97.79 142.24)
-		)
-		(stroke
-			(width 0)
-			(type default)
-		)
-	)
-	(wire
-		(pts
-			(xy 107.95 124.46) (xy 116.84 124.46)
 		)
 		(stroke
@@
 	)
 	(label "USB_D-"
-		(at 144.78 120.65 0)
+		(at 144.78 118.11 0)
 		(effects
 			(font
@@
 	)
 	(label "USB_D+"
-		(at 144.78 118.11 0)
-		(effects
-			(font
+		(at 144.78 120.65 0)
+		(effects
+			(font
