File: KICAD pcb/maibadge/maibadge_ver2.kicad_pcb (KiCad board)
At the start: 2 copper layers, 62.5 x 97.2 mm, 24 parts, among them J1 Conn_01x04_Socket, SW1 SW_Push, SW2 SW_Push, SW3 SW_Push, SW4 SW_Push, SW5 SW_Push, U1 ESP32-S3-WROOM-1, U10 SK6812SIDE-A-RVS, U2 AMS1117-3.3, U3 SK6812SIDE-A-RVS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

Commit message: feat: update pcb image
Parts:
- moved G*** 0.13 mm to (189.9, 86.5)

Commit message: feat: maibadge cab v2
Parts:
- removed SW2: SW_Push, Button_Switch_SMD:SW_Push_1P1T_XKB_TS-1187A
- added G***: LOGO, LOGO, B.Cu at (189.9, 93.5)
- added REF**: MountingHole_3.2mm_M3, MountingHole:MountingHole_3.2mm_M3, F.Cu at (165.2, 44.3)
- renumbered SW4 to BOOT, SW3 to RESET
Connections:
- J1 pad 2: /USB_D+ -> /USB_D-
- J1 pad 3: /USB_D- -> /USB_D+
Routing:
- net GND: track 28.2 -> 19.9 mm, vias 10 -> 8
- net /USB_D+: track 58.9 -> 65.3 mm, vias 2 -> 1
- net +3.3V: track 183.9 -> 177.7 mm
- net /button 1: track 51.3 -> 49.0 mm
- net /USB_D-: track 63.1 -> 64.6 mm, vias 2 -> 1
- net /main led DIN: track 64.3 -> 63.7 mm
Other:
- board text added: "maibadge cab by Justin and Terence"
